Commit message: multiview scanning

File: resources/ur3e/config/runtime_robot_description.urdf (robot description, URDF)
Before this commit: robot ur3e, 14 links, 13 joints
Links:
- added link hyperfusion_tcp; visual sphere radius=0.004
- link hyperfusion_tool_payload: mass 0.25 -> 0.35; geometry collision mesh filename=file:///mnt/d/Pototypy/HyperFusion/resources/ur3e/urdf/mesh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 scale=1 1 1; visual mesh filename=file:///mnt/d/Pototypy/HyperFusion/resources/ur3e/urdf/mesh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 scale=1 1 1
Joints:
- added joint tool0-hyperfusion_tcp: type fixed, parent tool0, child hyperfusion_tcp, origin xyz=0.000000 -0.056035 0.081825 rpy=0 0 0

File: resources/ur3e/srdf/hyperfusion_ur.srdf.xacro (robot description, xacro)
@@ -9,3 +9,6 @@
   <disable_collisions link1="flange" link2="hyperfusion_tool_payload" reason="Fixed"/>
   <disable_collisions link1="wrist_3_link" link2="hyperfusion_tool_payload" reason="Adjacent"/>
+  <disable_collisions link1="tool0" link2="hyperfusion_tcp" reason="Fixed"/>
+  <disable_collisions link1="flange" link2="hyperfusion_tcp" reason="Fixed"/>
+  <disable_collisions link1="hyperfusion_tool_payload" link2="hyperfusion_tcp" reason="Adjacent"/>
 </robot>

File: resources/ur3e/urdf/hyperfusion_tool_payload.xacro (robot description, xacro)
@@ -1,54 +1,75 @@
 <?xml version="1.0"?>
-<!-- Camera / sensor collision dome on tool0.
-     hemisphere: bowl on flange — apex at flange, flat rim opens outward (+tool0 Z).
-     sphere: full sphere centered on tool0. -->
+<!-- Camera / sensor collision payload on tool0.
+     mesh: real CAD STL (metres), flange-aligned — preferred.
+     hemisphere: legacy unit bowl scaled by radius_m.
+     sphere / box: simple primitives. -->
 <robot xmlns:xacro="http://wiki.ros.org/xacro">
   <xacro:macro name="hyperfusion_tool_payload"
-               params="tf_prefix shape radius_m box_x_m box_y_m box_z_m mesh_dir collision_gap_m origin_x_m origin_y_m origin_z_m origin_roll_rad origin_pitch_rad origin_yaw_rad">
+               params="tf_prefix shape radius_m box_x_m box_y_m box_z_m mesh_dir mesh_file collision_gap_m origin_x_m origin_y_m origin_z_m origin_roll_rad origin_pitch_rad origin_yaw_rad">
     <link name="${tf_prefix}hyperfusion_tool_payload">
       <visual name="hyperfusion_tool_payload_visual">
-        <!-- Hemisphere flipped 180° about X: apex at flange, flat rim faces outward (+tool0 Z). -->
-        <origin xyz="0 0 ${radius_m}" rpy="${pi} 0 0"/>
-        <geometry>
-          <xacro:if value="${shape == 'box'}">
-            <box size="${box_x_m} ${box_y_m} ${box_z_m}"/>
-          </xacro:if>
-          <xacro:if value="${shape == 'hemisphere'}">
+        <xacro:if value="${shape == 'mesh'}">
+          <!-- CAD was pan-180° off in tool0 XY → rotate about Z by π. -->
+          <origin xyz="0 0 0" rpy="0 0 ${pi}"/>
+          <geometry>
+            <mesh filename="file://${mesh_dir}${mesh_file}" scale="1 1 1"/>
+          </geometry>
+        </xacro:if>
+        <xacro:if value="${shape == 'hemisphere'}">
+          <!-- Unit bowl: apex at flange, flat rim opens +tool0 Z. -->
+          <origin xyz="0 0 ${radius_m}" rpy="${pi} 0 0"/>
+          <geometry>
             <mesh filename="file://${mesh_dir}tool_payload_hemisphere.stl"
                   scale="${radius_m} ${radius_m} ${radius_m}"/>
-          </xacro:if>
-          <xacro:if value="${shape == 'sphere'}">
+          </geometry>
+        </xacro:if>
+        <xacro:if value="${shape == 'box'}">
+          <origin xyz="0 0 0" rpy="0 0 0"/>
+          <geometry>
+            <box size="${box_x_m} ${box_y_m} ${box_z_m}"/>
+          </geometry>
+        </xacro:if>
+        <xacro:if value="${shape == 'sphere'}">
+          <origin xyz="0 0 0" rpy="0 0 0"/>
+          <geometry>
             <sphere radius="${radius_m}"/>
-          </xacro:if>
-        </geometry>
+          </geometry>
+        </xacro:if>
         <material name="hyperfusion_tool_payload_visual">
-          <color rgba="0.15 0.85 1.0 0.75"/>
+          <color rgba="0.15 0.85 1.0 0.55"/>
         </material>
       </visual>
       <collision>
-        <!-- Same flip; small +Z offset so MoveIt does not flag flange/wrist rim contact. -->
-        <origin xyz="0 0 ${radius_m + collision_gap_m}" rpy="${pi} 0 0"/>
-        <geometry>
-          <xacro:if value="${shape == 'box'}">
-            <box size="${box_x_m} ${box_y_m} ${box_z_m}"/>
-          </xacro:if>
-          <xacro:if value="${shape == 'hemisphere'}">
+        <xacro:if value="${shape == 'mesh'}">
+          <!-- CAD was pan-180° off in tool0 XY → rotate about Z by π. -->
+          <origin xyz="0 0 0" rpy="0 0 ${pi}"/>
+          <geometry>
+            <mesh filename="file://${mesh_dir}${mesh_file}" scale="1 1 1"/>
+          </geometry>
+        </xacro:if>
+        <xacro:if value="${shape == 'hemisphere'}">
+          <origin xyz="0 0 ${radius_m + collision_gap_m}" rpy="${pi} 0 0"/>
+          <geometry>
             <mesh filename="file://${mesh_dir}tool_payload_hemisphere.stl"
                   scale="${radius_m} ${radius_m} ${radius_m}"/>
-          </xacro:if>
-          <xacro:if value="${shape == 'sphere'}">
+          </geometry>
+        </xacro:if>
+        <xacro:if value="${shape == 'box'}">
+          <origin xyz="0 0 0" rpy="0 0 0"/>
+          <geometry>
+            <box size="${box_x_m} ${box_y_m} ${box_z_m}"/>
+          </geometry>
+        </xacro:if>
+        <xacro:if value="${shape == 'sphere'}">
+          <origin xyz="0 0 0" rpy="0 0 0"/>
+          <geometry>
             <sphere radius="${radius_m}"/>
-          </xacro:if>
-        </geometry>
+          </geometry>
+        </xacro:if>
       </collision>
       <inertial>
-        <xacro:if value="${shape == 'hemisphere'}">
-          <origin xyz="0 0 ${radius_m * 0.375}" rpy="0 0 0"/>
-        </xacro:if>
-        <xacro:unless value="${shape == 'hemisphere'}">
-          <origin xyz="0 0 0" rpy="0 0 0"/>
-        </xacro:unless>
-        <mass value="0.25"/>
-        <inertia ixx="0.0001" ixy="0" ixz="0" iyy="0.0001" iyz="0" izz="0.0001"/>
+        <origin xyz="0 0 0" rpy="0 0 0"/>
+        <mass value="0.35"/>
+        <inertia ixx="0.0002" ixy="0" ixz="0" iyy="0.0002" iyz="0" izz="0.0002"/>
       </inertial>
     </link>

File: resources/ur3e/urdf/hyperfusion_ur3e.urdf.xacro (robot description, xacro)
@@ -51,6 +51,6 @@
   <!-- Tool payload placeholder (camera / sensor envelope for MoveIt collision). -->
   <xacro:arg name="tool_payload_enabled" default="true"/>
-  <xacro:arg name="tool_payload_shape" default="hemisphere"/>
-  <xacro:arg name="tool_payload_radius_m" default="0.10"/>
+  <xacro:arg name="tool_payload_shape" default="mesh"/>
+  <xacro:arg name="tool_payload_radius_m" default="0.077"/>
   <xacro:arg name="tool_payload_box_x_m" default="0.08"/>
   <xacro:arg name="tool_payload_box_y_m" default="0.06"/>
@@ -59,9 +59,14 @@
   <xacro:arg name="tool_payload_y_m" default="0"/>
   <xacro:arg name="tool_payload_z_m" default="0"/>
-  <xacro:arg name="tool_payload_collision_gap_m" default="0.002"/>
+  <xacro:arg name="tool_payload_collision_gap_m" default="0.0"/>
   <xacro:arg name="tool_payload_mesh_dir" default="meshes/"/>
+  <xacro:arg name="tool_payload_mesh_file" default="ur_bfs_tool_payload.stl"/>
   <xacro:arg name="tool_payload_roll_rad" default="0"/>
   <xacro:arg name="tool_payload_pitch_rad" default="0"/>
   <xacro:arg name="tool_payload_yaw_rad" default="0"/>
+  <!-- Optical TCP (BFS sensor face centroid) in tool0 metres. -->
+  <xacro:arg name="tool_tcp_x_m" default="0"/>
+  <xacro:arg name="tool_tcp_y_m" default="-0.056035"/>
+  <xacro:arg name="tool_tcp_z_m" default="0.020"/>
   <xacro:property name="hf_pi" value="3.14159265358979323846"/>
   <xacro:property name="initial_positions_file" default="$(arg initial_positions_file)"/>
@@ -123,4 +128,5 @@
       radius_m="$(arg tool_payload_radius_m)"
       mesh_dir="$(arg tool_payload_mesh_dir)"
+      mesh_file="$(arg tool_payload_mesh_file)"
       collision_gap_m="$(arg tool_payload_collision_gap_m)"
       box_x_m="$(arg tool_payload_box_x_m)"
@@ -135,3 +141,20 @@
     />
   </xacro:if>
+  <!-- Scan / MoveIt tip: BFS sensor-face centroid (same +Z as tool0). -->
+  <link name="$(arg tf_prefix)hyperfusion_tcp">
+    <visual>
+      <origin xyz="0 0 0" rpy="0 0 0"/>
+      <geometry>
+        <sphere radius="0.004"/>
+      </geometry>
+      <material name="hyperfusion_tcp_marker">
+        <color rgba="1.0 0.25 0.1 0.95"/>
+      </material>
+    </visual>
+  </link>
+  <joint name="$(arg tf_prefix)tool0-hyperfusion_tcp" type="fixed">
+    <parent link="$(arg tf_prefix)tool0"/>
+    <child link="$(arg tf_prefix)hyperfusion_tcp"/>
+    <origin xyz="$(arg tool_tcp_x_m) $(arg tool_tcp_y_m) $(arg tool_tcp_z_m)" rpy="0 0 0"/>
+  </joint>
 </robot>

Commit message: 3d_scanning_stable

File: resources/ur3e/config/runtime_robot_description.urdf (robot description, URDF)
Before this commit: robot ur3e, 15 links, 14 joints
Joints:
- joint base_joint: origin xyz=0.000000 0.000000 0.600000 rpy=3.141593 0.000000 0.000000 -> xyz=0.000000 0.000000 0.640000 rpy=3.141593 0.000000 0.000000

Commit message: updated_payload_tool

File: resources/ur3e/config/runtime_robot_description.urdf (robot description, URDF)
Before this commit: robot ur3e, 15 links, 14 joints
Joints:
- joint base_joint: origin xyz=0.000000 0.000000 0.640000 rpy=3.141593 0.000000 0.000000 -> xyz=0.000000 0.000000 0.629000 rpy=3.141593 0.000000 0.000000
- joint tool0-hyperfusion_tcp: origin xyz=0.000000 -0.056035 0.081825 rpy=0 0 0 -> xyz=0.000715 -0.054197 0.073755 rpy=-0.03340211 0.01300270 0.00500560

File: resources/ur3e/urdf/hyperfusion_ur3e.urdf.xacro (robot description, xacro)
@@ -61,12 +61,15 @@
   <xacro:arg name="tool_payload_collision_gap_m" default="0.0"/>
   <xacro:arg name="tool_payload_mesh_dir" default="meshes/"/>
-  <xacro:arg name="tool_payload_mesh_file" default="ur_bfs_tool_payload.stl"/>
+  <xacro:arg name="tool_payload_mesh_file" default="ur_tool_payload.stl"/>
   <xacro:arg name="tool_payload_roll_rad" default="0"/>
   <xacro:arg name="tool_payload_pitch_rad" default="0"/>
   <xacro:arg name="tool_payload_yaw_rad" default="0"/>
-  <!-- Optical TCP (BFS sensor face centroid) in tool0 metres. -->
-  <xacro:arg name="tool_tcp_x_m" default="0"/>
-  <xacro:arg name="tool_tcp_y_m" default="-0.056035"/>
-  <xacro:arg name="tool_tcp_z_m" default="0.020"/>
+  <!-- Optical TCP (BFS optical origin) in tool0 metres + URDF rpy. Tsai hand-eye. -->
+  <xacro:arg name="tool_tcp_x_m" default="0.000715"/>
+  <xacro:arg name="tool_tcp_y_m" default="-0.054197"/>
+  <xacro:arg name="tool_tcp_z_m" default="0.073755"/>
+  <xacro:arg name="tool_tcp_roll_rad" default="-0.03340168"/>
+  <xacro:arg name="tool_tcp_pitch_rad" default="0.01300337"/>
+  <xacro:arg name="tool_tcp_yaw_rad" default="0.00500528"/>
   <xacro:property name="hf_pi" value="3.14159265358979323846"/>
   <xacro:property name="initial_positions_file" default="$(arg initial_positions_file)"/>
@@ -141,5 +144,5 @@
     />
   </xacro:if>
-  <!-- Scan / MoveIt tip: BFS sensor-face centroid (same +Z as tool0). -->
+  <!-- Scan / MoveIt tip: BFS optical origin (calibrated xyz + rpy vs tool0). -->
   <link name="$(arg tf_prefix)hyperfusion_tcp">
     <visual>
@@ -156,5 +159,6 @@
     <parent link="$(arg tf_prefix)tool0"/>
     <child link="$(arg tf_prefix)hyperfusion_tcp"/>
-    <origin xyz="$(arg tool_tcp_x_m) $(arg tool_tcp_y_m) $(arg tool_tcp_z_m)" rpy="0 0 0"/>
+    <origin xyz="$(arg tool_tcp_x_m) $(arg tool_tcp_y_m) $(arg tool_tcp_z_m)"
+            rpy="$(arg tool_tcp_roll_rad) $(arg tool_tcp_pitch_rad) $(arg tool_tcp_yaw_rad)"/>
   </joint>
 </robot>
