Commit message: Improve UR3e semi-ring reachability and FPP R400 scan plans.
Co-authored-by: Cursor <cursoragent@cursor.com>

File: app/sidecars/ur3e/config/runtime_p8767/runtime_robot_description.urdf (robot description, URDF)
Before this commit: robot ur3e, 15 links, 14 joints
Joints:
- joint tool0-hyperfusion_tcp: origin xyz=0.000715 -0.054197 0.073755 rpy=-0.03340211 0.01300270 0.00500560 -> xyz=0.000372 0.057104 0.027499 rpy=0.43633231 0.00000000 0.00000000

File: app/sidecars/ur3e/config/runtime_p8768/runtime_robot_description.urdf (robot description, URDF)
Before this commit: robot ur3e, 15 links, 14 joints
Joints:
- joint tool0-hyperfusion_tcp: origin xyz=0.000715 -0.054197 0.073755 rpy=-0.03340211 0.01300270 0.00500560 -> xyz=0.000372 0.057104 0.027499 rpy=0.43633231 0.00000000 0.00000000

File: app/sidecars/ur3e/config/runtime_robot_description.urdf (robot description, URDF)
Before this commit: robot ur3e, 15 links, 14 joints
Joints:
- joint base_joint: origin xyz=0.000000 0.000000 0.870000 rpy=3.141593 0.000000 0.000000 -> xyz=0.000000 0.000000 0.888000 rpy=3.141593 0.000000 0.000000
- joint tool0-hyperfusion_tcp: origin xyz=0.000715 -0.054197 0.073755 rpy=-0.03340211 0.01300270 0.00500560 -> xyz=0.000372 0.057104 0.027499 rpy=0.43633231 0.00000000 0.00000000
