Commit message: flat-reference calibration

File: app/sidecars/ur3e/config/runtime_robot_description.urdf (robot description, URDF)
Before this commit: robot ur3e, 15 links, 14 joints
Links:
- link hyperfusion_tool_payload: geometry collision mesh filename=file:///mnt/d/Pototypy/HyperFusion/app/sidecars/ur3e/urdf/m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 scale=1 1 1; visual mesh filename=file:///mnt/d/Pototypy/HyperFusion/app/sidecars/ur3e/urdf/m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 scale=1 1 1

Commit message: fpp_adjustment

File: app/sidecars/ur3e/config/runtime_robot_description.urdf (robot description, URDF)
Before this commit: robot ur3e, 15 links, 14 joints
Joints:
- joint base_joint: origin xyz=0.000000 0.000000 0.629000 rpy=3.141593 0.000000 0.000000 -> xyz=0.000000 0.000000 0.870000 rpy=3.141593 0.000000 0.000000

File: app/sidecars/ur3e/urdf/hyperfusion_ur3e.urdf.xacro (robot description, xacro)
@@ -61,5 +61,5 @@
   <xacro:arg name="tool_payload_collision_gap_m" default="0.0"/>
   <xacro:arg name="tool_payload_mesh_dir" default="meshes/"/>
-  <xacro:arg name="tool_payload_mesh_file" default="ur_tool_payload.stl"/>
+  <xacro:arg name="tool_payload_mesh_file" default="bfs_dlp_payload.stl"/>
   <xacro:arg name="tool_payload_roll_rad" default="0"/>
   <xacro:arg name="tool_payload_pitch_rad" default="0"/>

Commit message: mvs_recalibrated

File: app/sidecars/ur3e/config/runtime_robot_description.urdf (robot description, URDF)
Before this commit: robot ur3e, 15 links, 14 joints
Joints:
- joint base_joint: origin xyz=0.000000 0.000000 0.888000 rpy=3.141593 0.000000 0.000000 -> xyz=0.000000 0.000000 0.847500 rpy=3.141593 0.000000 0.000000
- joint tool0-hyperfusion_tcp: origin xyz=0.001400 0.031743 0.098538 rpy=-0.44092078 0.00418006 3.14039361 -> xyz=0.001993 0.038037 0.067403 rpy=-0.45881914 -0.00084125 -3.14997896
